Commit message: Update joint pos mode

File: sapien_env/sapien_env/assets/robot/panda/panda.urdf (robot description, URDF)
Before this commit: robot panda, 12 links, 11 joints
Links:
- added link panda_EE, mass 0.0
Joints:
- added joint panda_EE_joint: type fixed, parent panda_link8, child panda_EE, origin xyz=0 0 0.284 rpy=0 0 0, axis 0 0 0
